File: belamini_breakout_v01.brd (EAGLE design)
At the start: 71.1 x 105 mm, 112 parts, among them IC1 TL074D, IC10 LM4040B10, IC2 LM4041CIDBZ, IC3 TL074D, J1 M10SILK_FEMALE_PTH, SW1 EC12E_SW

Commit message: Swap output to line out
Parts:
- removed J4: (no value), SparkFun-Connectors:1X03
- moved R26 16.3 mm to (45.3, 26.3), turned to 270 degrees
- moved C14 1.90 mm to (35.7, 23.5), turned to 0 degrees
Connections:
- removed net L: J2.2
- removed net R: J2.3
- net DAC1: now also J2.2; no longer J4.3
- net DAC2: now also J2.1; no longer J4.2
- net GND: now also J2.3; no longer J2.1, J4.1
Routing:
- net N$24: track 6.22 -> 24.1 mm
- net DAC2: track 17.6 -> 11.2 mm
- net DAC1: track 13.8 -> 17.4 mm
- net D13: track 35.8 -> 32.9 mm
- net N$27: track 58.6 -> 57.3 mm
- net N$28: track 10.9 -> 10.3 mm
